File: Hardware/PCB/EPS&PAY/sources/PCB.kicad_sch (KiCad schematic)
At the start: 0 parts

Commit message: V0.1
Parts:
- added H1: PC/104 Connector, Connector_PinSocket_2.54mm:PinSocket_2x26_P2.54mm_Vertical, symbol Connector_Generic:Conn_02x26_Odd_Even
Connections:
- new net +5V: H1.16 (Pin_16), H1.20 (Pin_20), H1.24 (Pin_24), H1.28 (Pin_28), H1.32 (Pin_32), H1.36 (Pin_36)
- new net ADC_BAT: H1.44 (Pin_44)
- new net GND: H1.18 (Pin_18), H1.22 (Pin_22), H1.26 (Pin_26), H1.30 (Pin_30), H1.34 (Pin_34), H1.38 (Pin_38)
- no-connect marks 0 -> 39

Commit message: V0.2
Parts:
- added M1, M2, M3, M4: MountingHole, MountingHole:MountingHole_3.2mm_M3_Pad, symbol Mechanical:MountingHole
