File: Hardware/PCB/EPS&PAY/sources/PCB.kicad_pcb (KiCad board)
At the start: 4 copper layers, 87.2 x 77.2 mm, 141 parts, among them Q1 L8050, Q2 L8050, Q3 MMBTA06, SW1 SW_DPST_x2, SW2 SW_DPST_x2, U1 SCT2650STER, U10 TF_PUSH, U11 HX_TYPE-C_16PIN, U12 BH-18650-A1BJ021, U13 BWIPX-1-001E, U16 HX_TYPE-C_16PIN, U17 IP2326, U18 D2F, U19 AO4407A_C2841482, U2 AMS1117-3_3, U20 RASPBERRY_PI_4B_4GB, U3 AMS1117-3_3, U4 AMS1117-3_3, U5 ESP32-S3-WROOM-1-N4, U6 MPU-6050_C24112, U7 LIS3MDLTR, U8 LPS22HBTR, U9 DL-RFM95-915M

Commit message: V0.1
Parts:
- removed C17, C19, C20, C22, C23, C25, C26, C28, C29, C31, C32, C33, C34, C36, C53, C55, C6, C60, C7, C8: 100nF, EPS_PAY-Footprints:C0603
- removed C18, C30, C35, C39, C40, C59: 10uF, EPS_PAY-Footprints:C0805
- removed C21: 220pF, EPS_PAY-Footprints:C0603
- removed C24: 1uF, EPS_PAY-Footprints:C0805
- removed C51, C52, C54, C56, C57, C58: 1uF, EPS_PAY-Footprints:C0603
- removed D3, D6, D7: LED_GREEN, EPS_PAY-Footprints:LED0603-FD
- removed D4: SS34-MS, EPS_PAY-Footprints:DO-214AC_L4.3-W2.7-LS5.0-RD
- removed D5: USBLC6-2P6_C2827693, EPS_PAY-Footprints:SOT-666-6_L1.6-W1.2-P0.50-LS1.6-BL
- removed L3, L4, L5: 2.2nH, EPS_PAY-Footprints:L1008
- removed Q1, Q2: L8050, EPS_PAY-Footprints:SOT-23-3_L2.9-W1.3-P1.90-LS2.4-BR
- removed Q3: MMBTA06, EPS_PAY-Footprints:SOT-23-3_L2.9-W1.6-P1.90-LS2.8-BR
- removed R10, R6, R7, R8, R9: 1KΩ, EPS_PAY-Footprints:R0603
- removed R11, R16, R17, R30, R4, R5: 10KΩ, EPS_PAY-Footprints:R0603
- removed R12, R13, R14, R19, R20, R21, R22, R23, R24, R27, R28, R34, R35: 0Ω, EPS_PAY-Footprints:R0603
- removed R18: 10KΩ(NC), EPS_PAY-Footprints:R0603
- removed R25, R26, R36, R41, R45, R46, R47, R49: 5.1KΩ, EPS_PAY-Footprints:R0603
- removed R29: 56kΩ, EPS_PAY-Footprints:R0603
- removed SW1, SW2: SW_DPST_x2, EPS_PAY-Footprints:SW-SMD_L3.9-W3.0-P4.45
- removed U10: TF_PUSH, EPS_PAY-Footprints:TF-SMD_TF-PUSH
- removed U11: HX_TYPE-C_16PIN, EPS_PAY-Footprints:TYPE-C-SMD_HX-TYPE-C-16PIN
- removed U13: BWIPX-1-001E, EPS_PAY-Footprints:IPEX-SMD_BWIPX-1-001E
- removed U14: ~, GPS:GPS_NEO-M6
- removed U2, U3, U4: AMS1117-3_3, EPS_PAY-Footprints:SOT-223-3_L6.5-W3.4-P2.30-LS7.0-BR
- removed U20: RASPBERRY_PI_4B_4GB, RASPBERRY_PI_4B_4GB:MODULE_RASPBERRY_PI_4B_4GB
- removed U5: ESP32-S3-WROOM-1-N4, EPS_PAY-Footprints:WIFIM-SMD_ESP32-S3-WROOM-1-N8
- removed U6: MPU-6050_C24112, EPS_PAY-Footprints:QFN-24_L4.0-W4.0-P0.50-BL-EP2.7
- removed U7: LIS3MDLTR, EPS_PAY-Footprints:LGA-12_L2.0-W2.0-P0.50-BL
- removed U8: LPS22HBTR, EPS_PAY-Footprints:HLGA-10L_LPS22HBTR
- removed U9: DL-RFM95-915M, EPS_PAY-Footprints:LCC-16_L16.0-W16.0-P2.00-TL
- added H1: PC/104 Connector, Connector_PinSocket_2.54mm:PinSocket_2x26_P2.54mm_Vertical, F.Cu at (193.2, 45.0)
- C1, C13, C2, C3, C38, C4, C42, C43, C44, C45, C46, C47, C48, C49, C5, C50, C9, D1, D2, D8, D9, L1, L6, R1, R15, R2, R3, R31, R32, R33, R37, R38, R39, R40, R42, R43, R44, R48, R50, R51, R52, U1, U16, U17, U18, U19: moved to F.Cu
- moved R31 172.2 mm to (273.1, 93.5), turned to 0 degrees
- moved D9 169.6 mm to (268.0, 90.0), turned to 0 degrees
- moved D8 166.4 mm to (273.8, 89.2), turned to 0 degrees
- moved R52 162.2 mm to (272.4, 98.0), turned to 0 degrees
- moved R1 155.2 mm to (272.4, 95.9), turned to 0 degrees
- moved U17 151.9 mm to (260.1, 93.9)
- moved L6 149.5 mm to (253.6, 96.5)
- moved R33 149.5 mm to (253.7, 93.0), turned to 0 degrees
- moved U16 148.8 mm to (245.3, 86.3), turned to 0 degrees
- moved U1 146.8 mm to (260.7, 86.9), turned to 0 degrees
- moved D2 145.9 mm to (259.4, 98.6), turned to 0 degrees
- moved D1 143.9 mm to (268.0, 85.3), turned to 0 degrees
- moved L1 141.1 mm to (267.4, 95.5), turned to 0 degrees
- moved U19 138.0 mm to (254.2, 87.1), turned to 0 degrees
- moved R37 132.3 mm to (244.7, 94.6), turned to 0 degrees
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Routing:
- net +5V: track 229.1 -> 0.00 mm, vias 5 -> 0
- net /Carga Útil/ESP32_SLEEP_RPI: track 173.8 -> 0.00 mm
- net +3.3V_SEN: track 146.7 -> 0.00 mm, vias 1 -> 0
- net /Potência/BAT-: track 138.0 -> 0.00 mm
- net /Carga Útil/MOSI: track 132.9 -> 0.00 mm, vias 3 -> 0
- net /Carga Útil/SCK: track 126.5 -> 0.00 mm, vias 3 -> 0
- net /Potência/BATM: track 113.3 -> 0.00 mm, vias 1 -> 0
- net 8.4V: track 100.1 -> 0.00 mm, vias 2 -> 0
- net /Carga Útil/RPi5_TX_(UART2): track 88.8 -> 0.00 mm, vias 2 -> 0
- net /Carga Útil/RPi5_RX_(UART2): track 88.0 -> 0.00 mm, vias 2 -> 0
- net +3.3V ESP32: track 81.9 -> 0.00 mm, vias 4 -> 0
- net /Carga Útil/USB_DN: track 75.6 -> 0.00 mm
- net /Carga Útil/USB_DP: track 67.2 -> 0.00 mm
- net /Carga Útil/RESET: track 60.2 -> 0.00 mm, vias 2 -> 0
- net /Carga Útil/RPi5_GPS_TX_(UART1): track 53.4 -> 0.00 mm, vias 2 -> 0
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Other:
- board text removed: "BOOT"
- board text removed: "RESET"

Commit message: V0.2
Parts:
- added M1: MountingHole, MountingHole:MountingHole_3.2mm_M3_Pad, F.Cu at (95.7, 113.8)
- added M2: MountingHole, MountingHole:MountingHole_3.2mm_M3_Pad, F.Cu at (174.0, 114.2)
- added M3: MountingHole, MountingHole:MountingHole_3.2mm_M3_Pad, F.Cu at (96.0, 46.0)
- added M4: MountingHole, MountingHole:MountingHole_3.2mm_M3_Pad, F.Cu at (174.3, 45.1)
- added R36: 5.1KΩ, EPS_PAY-Footprints:R0603, F.Cu at (123.9, 71.0)
- added R41: 5.1KΩ, EPS_PAY-Footprints:R0603, F.Cu at (102.0, 70.6)
- added R49: 5.1KΩ, EPS_PAY-Footprints:R0603, F.Cu at (102.1, 64.7)
- moved D8 173.2 mm to (101.9, 67.9), turned to 90 degrees
- moved D9 170.9 mm to (100.1, 57.8), turned to -90 degrees
- moved R52 166.1 mm to (108.0, 74.6), turned to 90 degrees
- moved U17 154.9 mm to (108.3, 63.1), turned to -90 degrees
- moved D2 154.5 mm to (107.2, 71.8), turned to 180 degrees
- moved U16 150.1 mm to (96.4, 67.4), turned to -90 degrees
- moved L6 143.9 mm to (114.5, 59.7)
- moved R40 132.5 mm to (102.2, 72.9)
- moved R48 130.4 mm to (108.4, 69.1), turned to 90 degrees
- moved R38 130.4 mm to (104.7, 58.1)
- moved R39 128.8 mm to (106.2, 69.0), turned to 90 degrees
- moved R31 127.0 mm to (153.3, 51.3)
- moved R1 126.6 mm to (150.9, 60.2), turned to -90 degrees
- moved R37 126.0 mm to (121.7, 67.5)
- moved R42 125.4 mm to (110.2, 69.1), turned to 90 degrees
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Routing:
- net Net-(U1-SW): track 0.00 -> 10.8 mm
- net Net-(U1-GND): track 0.00 -> 5.22 mm
- removed copper zone on B.Cu, net GND
- removed copper zone on F.Cu, net GND
Other:
- copper layers 4 -> 2
- board text removed: "A antena tem um isolamnto mínimo de 15mm"
- board text removed: "Coloque vias para dissipação térmica de baixo dos CIs"
- board text removed: "Existe algum problema no meu ki-cad, em que, quando abre se recupera o arquivo em que os com footprint ficam na camada de user.coments"

Commit message: V0.3
Parts:
- moved C38 0.99 mm to (119.3, 58.7), turned to 90 degrees
- moved C1 0.46 mm to (170.7, 70.6)
- moved C2 0.46 mm to (171.2, 73.0)
- moved C50 0.46 mm to (170.2, 68.5)
- moved R36 0.23 mm to (123.8, 71.2)
Routing:
- net GND: track 0.00 -> 267.8 mm, vias 0 -> 6
- net 8.4V: track 0.00 -> 179.9 mm, vias 0 -> 6
- net /Potência/BATM: track 0.00 -> 123.6 mm, vias 0 -> 2
- net +5V: track 0.00 -> 93.8 mm
- net /Potência/BAT-: track 0.00 -> 87.1 mm, vias 0 -> 3
- net VIN: track 0.00 -> 36.0 mm
- net /Potência/n1: track 0.00 -> 29.7 mm, vias 0 -> 2
- net Net-(U17-NTC): track 0.00 -> 15.7 mm
- net /Potência/N_IP_1: track 0.00 -> 14.3 mm
- net Net-(U17-VSET): track 0.00 -> 12.0 mm
- net Net-(U17-VIN): track 0.00 -> 11.8 mm, vias 0 -> 2
- net Net-(U16-CC2): track 0.00 -> 9.02 mm, vias 0 -> 2
- net /Potência/DP: track 0.00 -> 8.79 mm
- net /Potência/P: track 0.00 -> 8.59 mm, vias 0 -> 2
- net Net-(C42-Pad1): track 0.00 -> 8.49 mm
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Other:
- board text removed: "Verificar lado do conector de bateria"

Commit message: Att: V0.4
Parts:
- U12: value BH-18650-A1BJ021 -> 1881561; footprint EPS_PAY-Footprints:BAT-TH_L77.0-W39.9_BH-18650-A1BJ021 -> EPS_PAY-Footprints:CONN-TH_3P-P2.50_C3585554
- moved U12 22.2 mm to (114.7, 90.1), turned to 90 degrees
Connections:
- C48 pad 1: /Potência/BAT- -> -8.4V
- C49 pad 1: /Potência/BAT- -> -8.4V
- R50 pad 2: 8.4V -> 8.4V_B
- U12 pad 3: /Potência/BATM -> -8.4V
- U17 pad 24: /Potência/BAT- -> -8.4V
- U19 pad 1: 8.4V -> 8.4V_B
- U19 pad 8: +5V -> 8.4V
Routing:
- net /Potência/BAT-: track 87.1 -> 0.00 mm, vias 3 -> 0
- net /Potência/BATM: track 123.6 -> 41.2 mm
- net -8.4V: track 0.00 -> 38.8 mm, vias 0 -> 3
- net 8.4V: track 179.9 -> 205.0 mm, vias 6 -> 4
- net +5V: track 93.8 -> 74.8 mm
- net 8.4V_B: track 0.00 -> 3.21 mm
