File: Hardware/PCB/EPS&PAY/sources/potencia.kicad_sch (KiCad schematic)
At the start: 50 parts, among them U1 SCT2650STER, U12 BH-18650-A1BJ021, U16 HX_TYPE-C_16PIN, U17 IP2326, U18 D2F, U19 AO4407A_C2841482

Commit message: Att: V0.4
Parts:
- removed U12: BH-18650-A1BJ021, EPS_PAY-Footprints:BAT-TH_L77.0-W39.9_BH-18650-A1BJ021, symbol EPS_PAY-Symbols:BH-18650-A1BJ021
- added U12: 1881561, EPS_PAY-Footprints:CONN-TH_3P-P2.50_C3585554, symbol EPS_PAY-Symbols:1881561
Connections:
- net +5V: no longer U19.8 (D)
- net 8.4V: now also U19.8 (D), U12.1; no longer R50.2, U19.1 (S)
- net BATM: now also U12.2
- net BAT- renamed -8.4V
- net -8.4V: now also U12.3
- new net 8.4V_B: R50.2, U19.1 (S)
Other:
- note removed: "Nova alteração"
